File: Single Tube Board/singleTube/singleTube.kicad_sch (KiCad schematic)
At the start: 42 parts, among them J1 USB_B_Micro, J2 Conn_01x04_Pin, Q1 BUT11, Q2 BUT11, SW1 SW_SPDT, U1 STM32F103C8T6, U2 NCH8200HV, U3 AMS1117-3.3, U5 K155ID1, Y1 16MHz, Y2 32.768KHz

Commit message: Finish routing single tube PCB
Parts:
- removed Q1, Q2: BUT11, Package_TO_SOT_THT:TO-220-3_Vertical, symbol Transistor_BJT:BUT11
- added Q1, Q2: MMBTA42, Package_TO_SOT_SMD:SOT-23, symbol Transistor_BJT:MMBTA42
Connections:
- net CONTROL_A: now also U1.16 (PA6); no longer U1.13 (PA3)
- net CONTROL_C: now also U1.13 (PA3); no longer U1.15 (PA5)
- net CONTROL_D: now also U1.15 (PA5); no longer U1.16 (PA6)
- net GND: now also Q1.2 (E), Q2.2 (E)
- net LHDP_C_T: now also Q2.1 (B)
- net LHDP_T_R: now also Q2.3 (C)
- net RHDP_C_T: now also Q1.1 (B)
- net RHDP_T_R: now also Q1.3 (C)
Changed lines of the file:
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@@
 		)
 	)
-	(label "CONTROL_D"
+	(label "CONTROL_A"
 		(at 210.82 60.96 0)
 		(effects
@@
 		)
 	)
-	(label "CONTROL_A"
+	(label "CONTROL_C"
 		(at 210.82 53.34 0)
 		(effects
@@
 		)
 	)
-	(label "CONTROL_C"
+	(label "CONTROL_D"
 		(at 210.82 58.42 0)
 		(effects
@@
 	)
 	(symbol
+		(lib_id "Transistor_BJT:MMBTA42")
+		(at 52.07 139.7 0)
+		(unit 1)
+		(body_style 1)
+		(exclude_from_sim no)
+		(in_bom yes)
+		(on_board yes)
+		(in_pos_files yes)
+		(dnp no)
+		(property "Reference" "Q2"
+			(at 57.15 138.4299 0)
+			(show_name no)
+			(do_not_autoplace no)
+			(effects
+				(font
+					(size 1.27 1.27)
+				)
+				(justify left)
+			)
+		)
+		(property "Value" "MMBTA42"
+			(at 57.15 140.9699 0)
+			(show_name no)
+			(do_not_autoplace no)
+			(effects
+				(font
+					(size 1.27 1.27)
+				)
+				(justify left)
+			)
+		)
+		(property "Footprint" "Package_TO_SOT_SMD:SOT-23"
+			(at 57.15 141.605 0)
+			(hide yes)
+			(show_name no)
+			(do_not_autoplace no)
+			(effects
+				(font
+					(size 1.27 1.27)
+					(italic yes)
+				)
+				(justify left)
+			)
+		)
+		(property "Datasheet" "https://www.onsemi.com/pub/Collateral/MMBTA42LT1-D.PDF"
+			(at 52.07 139.7 0)
+			(hide yes)
+			(show_name no)
+			(do_not_autoplace no)
+			(effects
+				(font
+					(size 1.27 1.27)
+				)
+				(justify left)
+			)
+		)
+		(property "Description" "0.5A Ic, 300V Vce, NPN High Voltage Transistor, SOT-23"
+			(at 52.07 139.7 0)
+			(hide yes)
+			(show_name no)
+			(do_not_autoplace no)
+			(effects
+				(font
+					(size 1.27 1.27)
+				)
+			)
+		)
+		(property "Sim.Device" "NPN"
+			(at 52.07 139.7 0)
+			(hide yes)
+			(show_name no)
+			(do_not_autoplace no)
+			(effects
+				(font
+					(size 1.27 1.27)
+				)
+			)
+		)
+		(property "Sim.Pins" "1=B 2=E 3=C"
+			(at 52.07 139.7 0)
+			(hide yes)
+			(show_name no)
+			(do_not_autoplace no)
+			(effects
+				(font
+					(size 1.27 1.27)
+				)
+			)
+		)
+		(pin "2"
+		)
+		(pin "1"
+		)
+		(pin "3"
+		)
+		(instances
+			(project "singleTube"
+				(path "/416fc244-fffc-4466-89c1-5a0f0bfc8b8d"
+					(reference "Q2")
+					(unit 1)
+				)
+			)
+		)
+	)
+	(symbol
 		(lib_id "Device:Crystal_GND24")
 		(at 110.49 58.42 0)
@@
 	)
 	(symbol
-		(lib_id "Transistor_BJT:BUT11")
-		(at 58.42 181.61 0)
-		(mirror y)
-		(unit 1)
-		(body_style 1)
-		(exclude_from_sim no)
-		(in_bom yes)
-		(on_board yes)
-		(in_pos_files yes)
-		(dnp no)
-		(property "Reference" "Q1"
-			(at 53.34 180.3399 0)
-			(show_name no)
-			(do_not_autoplace no)
-			(effects
-				(font
-					(size 1.27 1.27)
-				)
-				(justify left)
-			)
-		)
-		(property "Value" "BUT11"
-			(at 53.34 182.8799 0)
-			(show_name no)
-			(do_not_autoplace no)
-			(effects
-				(font
-					(size 1.27 1.27)
-				)
-				(justify left)
-			)
-		)
-		(property "Footprint" "Package_TO_SOT_THT:TO-220-3_Vertical"
-			(at 53.34 183.515 0)
-			(hide yes)
-			(show_name no)
-			(do_not_autoplace no)
-			(effects
-				(font
-					(size 1.27 1.27)
-					(italic yes)
-				)
-				(justify left)
-			)
-		)
-		(property "Datasheet" "https://www.onsemi.com/pub/Collateral/BUT11A-D.pdf"
-			(at 58.42 181.61 0)
-			(hide yes)
-			(show_name no)
-			(do_not_autoplace no)
-			(effects
-				(font
-					(size 1.27 1.27)
-				)
-				(justify left)
-			)
-		)
-		(property "Description" "5A Ic, 400V Vce, Silicon Power NPN Transistors, TO-220"
-			(at 58.42 181.61 0)
-			(hide yes)
-			(show_name no)
-			(do_not_autoplace no)
-			(effects
-				(font
-					(size 1.27 1.27)
-				)
-			)
-		)
-		(property "Sim.Device" "NPN"
-			(at 58.42 181.61 0)
-			(hide yes)
-			(show_name no)
-			(do_not_autoplace no)
-			(effects
-				(font
-					(size 1.27 1.27)
-				)
-			)
-		)
-		(property "Sim.Pins" "1=B 2=C 3=E"
-			(at 58.42 181.61 0)
-			(hide yes)
-			(show_name no)
-			(do_not_autoplace no)
-			(effects
-				(font
-					(size 1.27 1.27)
-				)
-			)
-		)
-		(pin "1"
-		)
-		(pin "2"
-		)
-		(pin "3"
-		)
-		(instances
-			(project "singleTube"
-				(path "/416fc244-fffc-4466-89c1-5a0f0bfc8b8d"
-					(reference "Q1")
-					(unit 1)
-				)
-			)
-		)
-	)
-	(symbol
 		(lib_id "Device:R")
 		(at 64.77 166.37 90)
@@
 	)
 	(symbol
+		(lib_id "Transistor_BJT:MMBTA42")
+		(at 58.42 181.61 0)
+		(mirror y)
+		(unit 1)
+		(body_style 1)
+		(exclude_from_sim no)
+		(in_bom yes)
+		(on_board yes)
+		(in_pos_files yes)
+		(dnp no)
+		(property "Reference" "Q1"
+			(at 53.34 180.3399 0)
+			(show_name no)
+			(do_not_autoplace no)
+			(effects
+				(font
+					(size 1.27 1.27)
+				)
+				(justify left)
+			)
+		)
+		(property "Value" "MMBTA42"
+			(at 53.34 182.8799 0)
+			(show_name no)
+			(do_not_autoplace no)
+			(effects
+				(font
+					(size 1.27 1.27)
+				)
+				(justify left)
+			)
+		)
+		(property "Footprint" "Package_TO_SOT_SMD:SOT-23"
+			(at 53.34 183.515 0)
+			(hide yes)
+			(show_name no)
+			(do_not_autoplace no)
+			(effects
+				(font
+					(size 1.27 1.27)
+					(italic yes)
+				)
+				(justify left)
+			)
+		)
+		(property "Datasheet" "https://www.onsemi.com/pub/Collateral/MMBTA42LT1-D.PDF"
+			(at 58.42 181.61 0)
+			(hide yes)
+			(show_name no)
+			(do_not_autoplace no)
+			(effects
+				(font
+					(size 1.27 1.27)
+				)
+				(justify left)
+			)
+		)
+		(property "Description" "0.5A Ic, 300V Vce, NPN High Voltage Transistor, SOT-23"
+			(at 58.42 181.61 0)
+			(hide yes)
+			(show_name no)
+			(do_not_autoplace no)
+			(effects
+				(font
+					(size 1.27 1.27)
+				)
+			)
+		)
+		(property "Sim.Device" "NPN"
+			(at 58.42 181.61 0)
+			(hide yes)
+			(show_name no)
+			(do_not_autoplace no)
+			(effects
+				(font
+					(size 1.27 1.27)
+				)
+			)
+		)
+		(property "Sim.Pins" "1=B 2=E 3=C"
+			(at 58.42 181.61 0)
+			(hide yes)
+			(show_name no)
+			(do_not_autoplace no)
+			(effects
+				(font
+					(size 1.27 1.27)
+				)
+			)
+		)
+		(pin "2"
+		)
+		(pin "1"
+		)
+		(pin "3"
+		)
+		(instances
+			(project "singleTube"
+				(path "/416fc244-fffc-4466-89c1-5a0f0bfc8b8d"
+					(reference "Q1")
+					(unit 1)
+				)
+			)
+		)
+	)
+	(symbol
 		(lib_id "nixie-project:NCH8200HV")
 		(at 33.02 154.94 0)
@@
 					(unit 1)
 				)
-			)
-		)
-	)
-	(symbol
-		(lib_id "Transistor_BJT:BUT11")
-		(at 52.07 139.7 0)
-		(unit 1)
-		(body_style 1)
-		(exclude_from_sim no)
-		(in_bom yes)
-		(on_board yes)
-		(in_pos_files yes)
-		(dnp no)
-		(property "Reference" "Q2"
-			(at 57.15 138.4299 0)
-			(show_name no)
-			(do_not_autoplace no)
-			(effects
-				(font
-					(size 1.27 1.27)
-				)
-				(justify left)
-			)
-		)
-		(property "Value" "BUT11"
-			(at 57.15 140.9699 0)
-			(show_name no)
-			(do_not_autoplace no)
-			(effects
-				(font
-					(size 1.27 1.27)
-				)
-				(justify left)
-			)
-		)
-		(property "Footprint" "Package_TO_SOT_THT:TO-220-3_Vertical"
-			(at 57.15 141.605 0)
-			(hide yes)
-			(show_name no)
-			(do_not_autoplace no)
-			(effects
-				(font
-					(size 1.27 1.27)
-					(italic yes)
-				)
-				(justify left)
-			)
-		)
-		(property "Datasheet" "https://www.onsemi.com/pub/Collateral/BUT11A-D.pdf"
-			(at 52.07 139.7 0)
-			(hide yes)
-			(show_name no)
-			(do_not_autoplace no)
-			(effects
-				(font
-					(size 1.27 1.27)
-				)
-				(justify left)
-			)
-		)
-		(property "Description" "5A Ic, 400V Vce, Silicon Power NPN Transistors, TO-220"
-			(at 52.07 139.7 0)
-			(hide yes)
-			(show_name no)
-			(do_not_autoplace no)
-			(effects
-				(font
-					(size 1.27 1.27)
-				)
-			)
-		)
-		(property "Sim.Device" "NPN"
-			(at 52.07 139.7 0)
-			(hide yes)
-			(show_name no)
-			(do_not_autoplace no)
-			(effects
-				(font
-					(size 1.27 1.27)
-				)
-			)
-		)
-		(property "Sim.Pins" "1=B 2=C 3=E"
-			(at 52.07 139.7 0)
-			(hide yes)
-			(show_name no)
-			(do_not_autoplace no)
-			(effects
-				(font
-					(size 1.27 1.27)
-				)
-			)
-		)
-		(pin "1"
-		)
-		(pin "2"
-		)
-		(pin "3"
-		)
-		(instances
-			(project "singleTube"
-				(path "/416fc244-fffc-4466-89c1-5a0f0bfc8b8d"
-					(reference "Q2")
-					(unit 1)
-				)

Commit message: Remove analog filtering, simplify routing
Parts:
- removed C6, C7: 1u, Capacitor_SMD:C_0402_1005Metric, symbol Device:C
- removed FB1: 120R, Inductor_SMD:L_0603_1608Metric, symbol Device:FerriteBead
- C8: value 10n -> 100n
Connections:
- net +3.3VA is gone; now on net +3.3V: C8.1, U1.9 (VDDA)

Commit message: Create BOM
Parts:
- C1, C2, C3, C4, C8, C9: JLCPCB Part # (none) -> C1525
- C10, C11: JLCPCB Part # (none) -> C1578
- C12, C13: JLCPCB Part # (none) -> C1554
- C14, C15: JLCPCB Part # (none) -> C45783
- C5: JLCPCB Part # (none) -> C19702
- D1: JLCPCB Part # (none) -> C2286
- J1: JLCPCB Part # (none) -> C397452
- J2: JLCPCB Part # (none) -> C5116483
- N1, U2, U5: now not fitted; now left out of the parts list
- Q1, Q2: JLCPCB Part # (none) -> C118557
- R1, R3: JLCPCB Part # (none) -> C25867
- R10, R7: JLCPCB Part # (none) -> C17999
- R11, R12: JLCPCB Part # (none) -> C17936
- R13: JLCPCB Part # (none) -> C17927
- R2: JLCPCB Part # (none) -> C25744
- R4: JLCPCB Part # (none) -> C17902
- SW1: JLCPCB Part # (none) -> C273395
- U1: JLCPCB Part # (none) -> C8734
- U3: JLCPCB Part # (none) -> C6186
- Y1: JLCPCB Part # (none) -> C13738
- Y2: JLCPCB Part # (none) -> C21547573
