File: Single Tube Board/singleTube/singleTube.kicad_pcb (KiCad board)
At the start: 2 copper layers, 49 x 68 mm, 42 parts, among them J1 USB_B_Micro, J2 Conn_01x04_Pin, Q1 BUT11, Q2 BUT11, SW1 SW_SPDT, U1 STM32F103C8T6, U2 NCH8200HV, U3 AMS1117-3.3, U5 K155ID1, Y1 16MHz, Y2 32.768KHz

Commit message: Finish routing single tube PCB
Parts:
- Q1, Q2: value BUT11 -> MMBTA42; footprint Package_TO_SOT_THT:TO-220-3_Vertical -> Package_TO_SOT_SMD:SOT-23
- moved Q2 16.9 mm to (68.8, 73.2)
- moved R12 13.5 mm to (73.5, 77.8)
- moved R7 13.5 mm to (73.0, 73.5)
- moved R10 11.6 mm to (73.7, 85.7)
- moved R11 11.6 mm to (74.7, 90.2)
- moved Q1 10.2 mm to (70.2, 87.2)
- moved C15 7.08 mm to (112.0, 82.8), turned to 90 degrees
- moved D1 3.78 mm to (112.5, 76.8), turned to -90 degrees
- moved R13 2.76 mm to (110.1, 110.6)
- moved R4 2.76 mm to (103.2, 115.5)
- moved U2 2.76 mm to (98.0, 104.2)
- moved U5 2.57 mm to (91.2, 86.5)
- moved C14 2.02 mm to (107.0, 76.5), turned to 0 degrees
- moved R3 1.82 mm to (112.0, 74.5), turned to 0 degrees
- moved U3 1.52 mm to (107.0, 82.2)
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Connections:
- Q1 pad 2: /RHDP_T_R -> GND
- Q1 pad 3: GND -> /RHDP_T_R
- Q2 pad 2: /LHDP_T_R -> GND
- Q2 pad 3: GND -> /LHDP_T_R
- U1 pad 13: /CONTROL_A -> /CONTROL_C
- U1 pad 15: /CONTROL_C -> /CONTROL_D
- U1 pad 16: /CONTROL_D -> /CONTROL_A
Routing:
- net +3.3V: track 9.25 -> 109.1 mm, vias 0 -> 4
- net /C3: track 0.00 -> 75.2 mm
- net /C7: track 0.00 -> 65.4 mm
- net /ANODE: track 0.00 -> 57.6 mm, vias 0 -> 2
- net /C6: track 0.00 -> 55.9 mm
- net /C4: track 0.00 -> 49.0 mm
- net GND: track 9.64 -> 56.5 mm, vias 0 -> 36
- net /C8: track 0.00 -> 44.4 mm
- net /C1: track 0.00 -> 42.7 mm, vias 0 -> 2
- net VBUS: track 0.00 -> 38.5 mm
- net /C9: track 0.00 -> 38.3 mm
- net /C2: track 0.00 -> 35.9 mm, vias 0 -> 2
- net /C5: track 0.00 -> 34.1 mm, vias 0 -> 2
- net /RHDP_CONTROL: track 0.00 -> 31.2 mm
- net /CLHDP: track 0.00 -> 28.3 mm
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- added copper zone on F.Cu, net +3.3V
- added copper zone on F.Cu, net /HV_R
- added copper zone on F.Cu, net GND
- added copper zone on F.Cu, net VBUS

Commit message: Remove analog filtering, simplify routing
Parts:
- removed C6, C7: 1u, Capacitor_SMD:C_0402_1005Metric
- removed FB1: 120R, Inductor_SMD:L_0603_1608Metric
- C8: value 10n -> 100n
Connections:
- C8 pad 1: +3.3VA -> +3.3V
- U1 pad 9: +3.3VA -> +3.3V
Routing:
- net +3.3VA: track 7.03 -> 0.00 mm
- net +3.3V: track 109.1 -> 116.1 mm
- net GND: track 56.5 -> 54.4 mm, vias 36 -> 34

Commit message: Remove unnecessary ground vias
Routing:
- net GND: track 54.4 -> 45.0 mm, vias 34 -> 30
Changed lines of the file:
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@@
-	)
-	(segment
-		(start 89.98 90.31)
-		(end 89.98 88.02)
-		(width 0.5)
-		(layer "F.Cu")
-		(net "GND")
 	)
 	(segment
@@
 	)
 	(segment
-		(start 86.5 59.5)
-		(end 84.5 59.5)
-		(width 0.5)
-		(layer "F.Cu")
-		(net "GND")
-	)
-	(segment
 		(start 110.095 109.0925)
 		(end 111.6575 109.0925)
@@
 	)
 	(segment
-		(start 97.746 96.754)
-		(end 95.75 98.75)
-		(width 0.5)
-		(layer "F.Cu")
-		(net "GND")
-	)
-	(segment
 		(start 100.6625 68.25)
 		(end 99.25 68.25)
@@
 	)
 	(segment
-		(start 89.98 88.02)
-		(end 90 88)
-		(width 0.5)
-		(layer "F.Cu")
-		(net "GND")
-	)
-	(segment
 		(start 111.5 75)
 		(end 111.25 75.25)
@@
 	)
 	(segment
-		(start 92.666 111.334)
-		(end 94.25 109.75)
-		(width 0.5)
-		(layer "F.Cu")
-		(net "GND")
-	)
-	(segment
 		(start 97.746 96.63)
 		(end 97.746 96.754)
@@
 	)
 	(via
-		(at 94.25 109.75)
-		(size 0.7)
-		(drill 0.3)
-		(layers "F.Cu" "B.Cu")
-		(net "GND")
-	)
-	(via
 		(at 98.5 73.25)
 		(size 0.7)
@@
 	)
 	(via
-		(at 95.75 98.75)
-		(size 0.7)
-		(drill 0.3)
-		(layers "F.Cu" "B.Cu")
-		(net "GND")
-	)
-	(via
 		(at 90.5 65.75)
 		(size 0.7)
@@
 		(layers "F.Cu" "B.Cu")
 		(free yes)
-		(net "GND")
-	)
-	(via
-		(at 84.5 59.5)
-		(size 0.7)
-		(drill 0.3)
-		(layers "F.Cu" "B.Cu")
-		(net "GND")
-	)
-	(via
-		(at 90 88)
-		(size 0.7)
-		(drill 0.3)
-		(layers "F.Cu" "B.Cu")
 		(net "GND")
 	)
@@
 	)
 	(segment
-		(start 75.2375 86.0625)
-		(end 78.3 83)
+		(start 73.83505 88.2875)
+		(end 74.5625 89.01495)
 		(width 0.3)
 		(layer "F.Cu")
@@
 	)
 	(segment
-		(start 77.7231 98.069185)
-		(end 77.7231 94.96305)
+		(start 72.786505 103.00578)
+		(end 70.35574 103.00578)
 		(width 0.3)
 		(layer "F.Cu")
@@
 	)
 	(segment
-		(start 77.7231 94.96305)
-		(end 74.5625 91.802449)
+		(start 72.749202 88.2875)
+		(end 73.83505 88.2875)
 		(width 0.3)
 		(layer "F.Cu")
@@
 	)
 	(segment
-		(start 74.5625 91.802449)
-		(end 74.5625 89.01495)
+		(start 72.749202 86.0625)
+		(end 72.2875 86.524202)
 		(width 0.3)
 		(layer "F.Cu")
@@
 	)
 	(segment
-		(start 72.2875 86.524202)
-		(end 72.749202 86.0625)
-		(width 0.3)
-		(layer "F.Cu")
-		(net "/C2")
-	)
-	(segment
-		(start 74.5625 89.01495)
-		(end 73.83505 88.2875)
-		(width 0.3)
-		(layer "F.Cu")
-		(net "/C2")
-	)
-	(segment
-		(start 73.83505 88.2875)
+		(start 72.2875 87.825798)
 		(end 72.749202 88.2875)
-		(width 0.3)
-		(layer "F.Cu")
-		(net "/C2")
-	)
-	(segment
-		(start 72.749202 88.2875)
-		(end 72.2875 87.825798)
-		(width 0.3)
-		(layer "F.Cu")
-		(net "/C2")
-	)
-	(segment
-		(start 79.9 83)
-		(end 82.05 83)
-		(width 0.3)
-		(layer "F.Cu")
-		(net "/C2")
-	)
-	(segment
-		(start 78.3 83)
-		(end 78.1 83)
-		(width 0.3)
-		(layer "F.Cu")
-		(net "/C2")
-	)
-	(segment
-		(start 72.749202 86.0625)
-		(end 75.2375 86.0625)
-		(width 0.3)
-		(layer "F.Cu")
-		(net "/C2")
-	)
-	(segment
-		(start 72.2875 87.825798)
-		(end 72.2875 86.524202)
 		(width 0.3)
 		(layer "F.Cu")
@@
 	)
 	(segment
-		(start 72.786505 103.00578)
+		(start 77.7231 98.069185)
+		(end 72.786505 103.00578)
+		(width 0.3)
+		(layer "F.Cu")
+		(net "/C2")
+	)
+	(segment
+		(start 74.5625 89.01495)
+		(end 74.5625 91.802449)
+		(width 0.3)
+		(layer "F.Cu")
+		(net "/C2")
+	)
+	(segment
+		(start 75.2375 86.0625)
+		(end 72.749202 86.0625)
+		(width 0.3)
+		(layer "F.Cu")
+		(net "/C2")
+	)
+	(segment
+		(start 79.7 83)
+		(end 82.05 83)
+		(width 0.3)
+		(layer "F.Cu")
+		(net "/C2")
+	)
+	(segment
+		(start 77.7231 94.96305)
 		(end 77.7231 98.069185)
 		(width 0.3)
@@
 	)
 	(segment
-		(start 70.35574 103.00578)
-		(end 72.786505 103.00578)
+		(start 74.5625 91.802449)
+		(end 77.7231 94.96305)
 		(width 0.3)
 		(layer "F.Cu")
 		(net "/C2")
 	)
-	(via
-		(at 78.1 83)
-		(size 0.7)
-		(drill 0.3)
-		(layers "F.Cu" "B.Cu")
+	(segment
+		(start 72.2875 86.524202)
+		(end 72.2875 87.825798)
+		(width 0.3)
+		(layer "F.Cu")
 		(net "/C2")
 	)
-	(via
-		(at 79.9 83)
-		(size 0.7)
-		(drill 0.3)
-		(layers "F.Cu" "B.Cu")
+	(segment
+		(start 78.3 83)
+		(end 75.2375 86.0625)
+		(width 0.3)
+		(layer "F.Cu")
 		(net "/C2")
 	)
-	(segment
-		(start 78.1 83)
-		(end 79.9 83)
+	(via
+		(at 78.3 83)
+		(size 0.7)
+		(drill 0.3)
+		(layers "F.Cu" "B.Cu")
+		(net "/C2")
+	)
+	(via
+		(at 79.7 83)
+		(size 0.7)
+		(drill 0.3)
+		(layers "F.Cu" "B.Cu")
+		(net "/C2")
+	)
+	(segment
+		(start 78.3 83)
+		(end 79.7 83)
 		(width 0.3)
 		(layer "B.Cu")

Commit message: Create BOM
Parts:
- added G***: LOGO, LOGO, F.Cu at (85.5, 116.0)
Other:
- board text added: "Aadit M."
- board text added: "BOOT"
- board text added: "June-July 2026 (6-7)"
- board text added: "SWD"
- board text added: "v0.1"
Changed lines of the file:
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@@
 		(embedded_fonts no)
 	)
+	(footprint "LOGO"
+		(layer "F.Cu")
+		(at 85.5 116)
+		(property "Reference" "G***"
+			(at 0 0 0)
+			(layer "F.SilkS")
+			(hide yes)
+			(effects
+				(font
+					(size 1.5 1.5)
+					(thickness 0.3)
+				)
+			)
+		)
+		(property "Value" "LOGO"
+			(at 0.75 0 0)
+			(layer "F.SilkS")
+			(hide yes)
+			(effects
+				(font
+					(size 1.5 1.5)
+					(thickness 0.3)
+				)
+			)
+		)
+		(property "Datasheet" ""
+			(at 0 0 0)
+			(layer "F.Fab")
+			(hide yes)
+			(effects
+				(font
+					(size 1.27 1.27)
+				)
+			)
+		)
+		(property "Description" ""
+			(at 0 0 0)
+			(layer "F.Fab")
+			(hide yes)
+			(effects
+				(font
+					(size 1.27 1.27)
+				)
+			)
+		)
+		(attr board_only exclude_from_pos_files exclude_from_bom)
+		(duplicate_pad_numbers_are_jumpers no)
+		(fp_poly
+			(pts
+				(xy -0.383966 -3.248092) (xy -0.313246 -3.229613) (xy -0.256633 -3.23608) (xy -0.131034 -3.227169)
+				(xy 0.023229 -3.142301) (xy 0.206052 -2.98154) (xy 0.246847 -2.939429) (xy 0.398554 -2.77492) (xy 0.513567 -2.635587)
+				(xy 0.606505 -2.498744) (xy 0.691986 -2.341709) (xy 0.784629 -2.141796) (xy 0.834158 -2.02807) (xy 0.924982 -1.82861)
+				(xy 1.020221 -1.638384) (xy 1.107914 -1.480291) (xy 1.170068 -1.384977) (xy 1.259206 -1.246765)
+				(xy 1.286085 -1.146585) (xy 1.282105 -1.120817) (xy 1.246748 -0.987507) (xy 1.236862 -0.891059)
+				(xy 1.259415 -0.807695) (xy 1.321371 -0.713636) (xy 1.429697 -0.585103) (xy 1.443764 -0.56896) (xy 1.594645 -0.391437)
+				(xy 1.720913 -0.229283) (xy 1.827514 -0.071015) (xy 1.919398 0.094854) (xy 2.00151 0.279808) (xy 2.078798 0.495331)
+				(xy 2.156209 0.75291) (xy 2.23869 1.064029) (xy 2.33119 1.440173) (xy 2.358669 1.554979) (xy 2.414256 1.826326)
+				(xy 2.457115 2.112326) (xy 2.485871 2.394645) (xy 2.499152 2.654952) (xy 2.495583 2.874912) (xy 2.473792 3.036194)
+				(xy 2.470552 3.048409) (xy 2.421588 3.139925) (xy 2.326064 3.21351) (xy 2.174819 3.273016) (xy 1.95869 3.322294)
+				(xy 1.738491 3.3562) (xy 1.529746 3.38562) (xy 1.328226 3.416783) (xy 1.160941 3.445372) (xy 1.07696 3.461916)
+				(xy 0.929175 3.486278) (xy 0.742227 3.506198) (xy 0.56896 3.51679) (xy 0.393165 3.525657) (xy 0.171569 3.541037)
+				(xy -0.060858 3.560364) (xy -0.18288 3.571971) (xy -0.386231 3.592287) (xy -0.527018 3.604837) (xy -0.62359 3.609594)
+				(xy -0.694296 3.606533) (xy -0.757482 3.595628) (xy -0.831496 3.576854) (xy -0.85344 3.571034) (xy -0.972285 3.544801)
+				(xy -1.131548 3.516102) (xy -1.253944 3.497325) (xy -1.462999 3.445399) (xy -1.678116 3.354182)
+				(xy -1.872389 3.237873) (xy -2.018908 3.110672) (xy -2.043588 3.080619) (xy -2.077607 3.026316)
+				(xy -2.095093 2.963606) (xy -2.097304 2.872428) (xy -2.085501 2.732719) (xy -2.072525 2.619835)
+				(xy -2.058928 2.471816) (xy -2.045103 2.259894) (xy -2.031894 2.001439) (xy -2.020144 1.713819)
+				(xy -2.010697 1.414406) (xy -2.007417 1.28016) (xy -1.998517 0.924049) (xy -1.987447 0.63753) (xy -1.971542 0.408913)
+				(xy -1.948139 0.226511) (xy -1.914575 0.078635) (xy -1.868187 -0.046402) (xy -1.80631 -0.160288)
+				(xy -1.726282 -0.274711) (xy -1.625439 -0.401359) (xy -1.623778 -0.403383) (xy -1.504178 -0.554463)
+				(xy -1.433102 -0.660064) (xy -1.403026 -0.733572) (xy -1.406426 -0.788375) (xy -1.406817 -0.789463)
+				(xy -1.427757 -0.901213) (xy -1.436977 -1.076028) (xy -1.435892 -1.268868) (xy -0.69088 -1.268868)
+				(xy -0.69088 -1.268471) (xy -0.681005 -1.198525) (xy -0.640546 -1.159103) (xy -0.553258 -1.143659)
+				(xy -0.402892 -1.14565) (xy -0.387748 -1.146362) (xy -0.250479 -1.156294) (xy -0.176139 -1.173812)
+				(xy -0.146377 -1.205879) (xy -0.14224 -1.23952) (xy -0.15112 -1.283369) (xy -0.189445 -1.309618)
+				(xy -0.274744 -1.324229) (xy -0.41656 -1.332817) (xy -0.56282 -1.336918) (xy -0.645601 -1.330369)
+				(xy -0.682441 -1.309057) (xy -0.69088 -1.268868) (xy -1.435892 -1.268868) (xy -1.435735 -1.296733)
+				(xy -1.425287 -1.546157) (xy -1.408381 -1.785995) (xy -1.298737 -1.785995) (xy -1.28122 -1.702652)
+				(xy -1.21468 -1.632209) (xy -1.12888 -1.578626) (xy -1.21468 -1.518529) (xy -1.284382 -1.444407)
+				(xy -1.2957 -1.373596) (xy -1.24968 -1.330223) (xy -1.172278 -1.333042) (xy -1.062438 -1.369371)
+				(xy -0.945903 -1.426123) (xy -0.848414 -1.490214) (xy -0.795711 -1.548557) (xy -0.79248 -1.562643)
+				(xy -0.825474 -1.619382) (xy -0.908598 -1.691482) (xy -1.018064 -1.764281) (xy -1.130086 -1.823117)
+				(xy -1.220876 -1.853329) (xy -1.258552 -1.849917) (xy -1.298737 -1.785995) (xy -1.408381 -1.785995)
+				(xy -1.406891 -1.807126) (xy -1.381804 -2.062466) (xy -1.351282 -2.295005) (xy -1.316583 -2.48757)
+				(xy -1.278964 -2.622987) (xy -1.271246 -2.6416) (xy -1.149433 -2.841572) (xy -0.983308 -3.020524)
+				(xy -0.794772 -3.158532) (xy -0.622756 -3.231593) (xy -0.500477 -3.254709) (xy -0.409489 -3.256604)
+			)
+			(stroke
+				(width 0)
+				(type solid)
+			)
+			(fill yes)
+			(layer "F.SilkS")
+		)
+		(embedded_fonts no)
+	)
 	(footprint "Connector_PinHeader_2.54mm:PinHeader_1x04_P2.54mm_Vertical"
 		(layer "F.Cu")
@@
 		(tags "capacitor")
 		(property "Reference" "C14"
-			(at 0 -1.75 0)
+			(at -3.25 0 0)
 			(layer "F.SilkS")
 			(effects
@@
 		(tags "capacitor")
 		(property "Reference" "C12"
-			(at 1.77 0.25 180)
+			(at 1.77 0.5 180)
 			(layer "F.SilkS")
 			(effects
@@
 		(property "Reference" "SW1"
 			(at 13 -2.5 180)
-			(layer "F.SilkS")
+			(layer "F.Fab")
 			(effects
 				(font
@@
 		(tags "capacitor")
 		(property "Reference" "C4"
-			(at -0.02 -1.5 180)
+			(at -1.5 0 180)
 			(layer "F.SilkS")
 			(effects
@@
 		(tags "resistor")
 		(property "Reference" "R3"
-			(at -2.01 0.25 0)
+			(at -2.01 0 0)
 			(layer "F.SilkS")
 			(effects
@@
 		(layer "Edge.Cuts")
 	)
+	(gr_text "BOOT"
+		(at 75.25 64.25 0)
+		(layer "F.SilkS")
+		(effects
+			(font
+				(size 1 1)
+				(thickness 0.1)
+			)
+			(justify left bottom)
+		)
+	)
+	(gr_text "SWD"
+		(at 96.75 57 0)
+		(layer "F.SilkS")
+		(effects
+			(font
+				(size 1 1)
+				(thickness 0.1)
+			)
+			(justify left bottom)
+		)
+	)
+	(gr_text "June-July 2026\n(6-7)"
+		(at 68.25 67.5 0)
+		(layer "B.SilkS")
+		(effects
+			(font
+				(size 1 1)
+				(thickness 0.2)
+				(bold yes)
+			)
+			(justify right bottom mirror)
+		)
+	)
+	(gr_text "v0.1"
+		(at 68.5 70.25 0)
+		(layer "B.SilkS")
+		(effects
+			(font
+				(size 1 1)
+				(thickness 0.2)
+				(bold yes)
+			)
+			(justify right bottom mirror)
+		)
+	)
+	(gr_text "Aadit M."
+		(at 68.5 72.75 0)
+		(layer "B.SilkS")
+		(effects
+			(font
+				(size 1 1)
+				(thickness 0.2)
+				(bold yes)
+			)
+			(justify right bottom mirror)
+		)
+	)
 	(segment

Commit message: update manufacturing files for single tube board
Other:
- board text removed: "Aadit M."
Changed lines of the file:
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@@
 			(usegerberattributes yes)
 			(usegerberadvancedattributes yes)
-			(creategerberjobfile yes)
+			(creategerberjobfile no)
 			(dashed_line_dash_ratio 12)
 			(dashed_line_gap_ratio 3)
@@
 			(crossoutdnponfab yes)
 			(subtractmaskfromsilk no)
-			(outputformat 1)
+			(outputformat 4)
 			(mirror no)
-			(drillshape 1)
+			(drillshape 0)
 			(scaleselection 1)
-			(outputdirectory "")
+			(outputdirectory "documents/")
 		)
 	)
@@
 		(property "Reference" "SW1"
 			(at 13 -2.5 180)
-			(layer "F.Fab")
+			(layer "F.SilkS")
 			(effects
 				(font
@@
 		)
 	)
-	(gr_text "Aadit M."
+	(gr_text "v0.1"
 		(at 68.5 72.75 0)
 		(layer "B.SilkS")
@@
 	)
 	(segment
-		(start 95.25 82.5)
-		(end 95.06 82.69)
+		(start 87.75 79.5)
+		(end 84.9 82.35)
 		(width 0.3)
 		(layer "F.Cu")
-		(net "/CONTROL_A")
+		(net "/CONTROL_C")
 	)
 	(segment
-		(start 95.25 74.6625)
-		(end 95.25 82.5)
+		(start 93.75 74.6625)
+		(end 93.75 78.5)
 		(width 0.3)
 		(layer "F.Cu")
-		(net "/CONTROL_A")
+		(net "/CONTROL_C")
+	)
+	(segment
+		(start 93.75 78.5)
+		(end 92.75 79.5)
+		(width 0.3)
+		(layer "F.Cu")
+		(net "/CONTROL_C")
+	)
+	(segment
+		(start 92.75 79.5)
+		(end 87.75 79.5)
+		(width 0.3)
+		(layer "F.Cu")
+		(net "/CONTROL_C")
+	)
+	(segment
+		(start 84.9 82.35)
+		(end 84.9 82.69)
+		(width 0.3)
+		(layer "F.Cu")
+		(net "/CONTROL_C")
 	)
 	(segment
@@
 	)
 	(segment
-		(start 87.75 79.5)
-		(end 84.9 82.35)
-		(width 0.3)
-		(layer "F.Cu")
-		(net "/CONTROL_C")
-	)
-	(segment
-		(start 93.75 74.6625)
-		(end 93.75 78.5)
-		(width 0.3)
-		(layer "F.Cu")
-		(net "/CONTROL_C")
-	)
-	(segment
-		(start 93.75 78.5)
-		(end 92.75 79.5)
-		(width 0.3)
-		(layer "F.Cu")
-		(net "/CONTROL_C")
-	)
-	(segment
-		(start 92.75 79.5)
-		(end 87.75 79.5)
+		(start 94.75 80.46)
+		(end 92.52 82.69)
 		(width 0.3)
 		(layer "F.Cu")
-		(net "/CONTROL_C")
+		(net "/CONTROL_D")
 	)
 	(segment
-		(start 84.9 82.35)
-		(end 84.9 82.69)
+		(start 94.75 74.6625)
+		(end 94.75 80.46)
 		(width 0.3)
 		(layer "F.Cu")
-		(net "/CONTROL_C")
+		(net "/CONTROL_D")
 	)
 	(segment
-		(start 94.75 80.46)
-		(end 92.52 82.69)
+		(start 95.25 82.5)
+		(end 95.06 82.69)
 		(width 0.3)
 		(layer "F.Cu")
-		(net "/CONTROL_D")
+		(net "/CONTROL_A")
 	)
 	(segment
-		(start 94.75 74.6625)
-		(end 94.75 80.46)
+		(start 95.25 74.6625)
+		(end 95.25 82.5)
 		(width 0.3)
 		(layer "F.Cu")
-		(net "/CONTROL_D")
+		(net "/CONTROL_A")
 	)
 	(segment
@@
 	)
 	(segment
-		(start 72.6875 90.8125)
-		(end 71.24755 90.8125)
-		(width 0.3)
-		(layer "F.Cu")
-		(net "/RHDP_C_T")
-	)
-	(segment
-		(start 71.24755 90.8125)
-		(end 69.2625 88.82745)
-		(width 0.3)
-		(layer "F.Cu")
-		(net "/RHDP_C_T")
-	)
-	(segment
-		(start 73.25 90.25)
-		(end 72.6875 90.8125)
+		(start 72.7625 72.3125)
+		(end 73.0375 72.0375)
 		(width 0.3)
 		(layer "F.Cu")
-		(net "/RHDP_C_T")
+		(net "/LHDP_T_R")
 	)
 	(segment
-		(start 69.2625 88.82745)
-		(end 69.2625 88.1875)
+		(start 68.7875 72.3125)
+		(end 72.7625 72.3125)
 		(width 0.3)
 		(layer "F.Cu")
-		(net "/RHDP_C_T")
+		(net "/LHDP_T_R")
 	)
 	(segment
@@
 	)
 	(segment
-		(start 72.7625 72.3125)
-		(end 73.0375 72.0375)
+		(start 72.6875 90.8125)
+		(end 71.24755 90.8125)
 		(width 0.3)
 		(layer "F.Cu")
-		(net "/LHDP_T_R")
+		(net "/RHDP_C_T")
 	)
 	(segment
-		(start 68.7875 72.3125)
-		(end 72.7625 72.3125)
+		(start 71.24755 90.8125)
+		(end 69.2625 88.82745)
 		(width 0.3)
 		(layer "F.Cu")
-		(net "/LHDP_T_R")
+		(net "/RHDP_C_T")
+	)
+	(segment
+		(start 73.25 90.25)
+		(end 72.6875 90.8125)
+		(width 0.3)
+		(layer "F.Cu")
+		(net "/RHDP_C_T")
+	)
+	(segment
+		(start 69.2625 88.82745)
+		(end 69.2625 88.1875)
+		(width 0.3)
+		(layer "F.Cu")
+		(net "/RHDP_C_T")
 	)
 	(zone
